Commit message: 032: add LeFranX adapter mount to fr3_xhand (roll-90, yaw-45 / clock315), palm-down

File: assets/urdf/fr3_xhand_description/fr3_xhand/fr3_xhand.urdf (robot description, URDF)
Before this commit: robot fr3_xhand, 22 links, 21 joints
Joints:
- joint hand_mount: origin xyz=0 0 0 rpy=0 0 3.14159 -> xyz=-0.017 -0.017 0.051 rpy=-1.5708 0 -0.7854
