Commit message: 008: rebuild fr3_xhand URDF from official XHand1 v1.3
Graft the official hand subtree (5 tip pads, per-link inertials summing to
1.1 kg, real effort caps 1.1/0.4 Nm), renamed to the existing joint/link
names so scene_utils is unchanged. Spawn-validated at 19 DoF; grasp pre-flight
closes, holds, and lifts a block 4/4 envs.

Co-Authored-By: Claude Opus 4.8 (1M context) <noreply@anthropic.com>

File: assets/urdf/fr3_xhand_description/fr3_xhand/fr3_xhand.urdf (robot description, URDF)
Before this commit: robot fr3_xhand, 22 links, 21 joints
Links:
- added link back_link, mass 0.00000002; collision mesh filename=/home/nas_main/sibeenkim/work/simtoolreal/assets/urdf/fr3_x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; visual mesh filename=/home/nas_main/sibeenkim/work/simtoolreal/assets/urdf/fr3_x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
- added link ee_link, mass 0.00000565; collision mesh filename=/home/nas_main/sibeenkim/work/simtoolreal/assets/urdf/fr3_x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; visual mesh filename=/home/nas_main/sibeenkim/work/simtoolreal/assets/urdf/fr3_x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
- added link index_rota_tip, mass 0.00000565; collision mesh filename=/home/nas_main/sibeenkim/work/simtoolreal/assets/urdf/fr3_x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; visual mesh filename=/home/nas_main/sibeenkim/work/simtoolreal/assets/urdf/fr3_x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
- added link index_rotaback_link1, mass 0.00000002; collision mesh filename=/home/nas_main/sibeenkim/work/simtoolreal/assets/urdf/fr3_x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; visual mesh filename=/home/nas_main/sibeenkim/work/simtoolreal/assets/urdf/fr3_x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
- added link index_rotaback_link2, mass 0.00000001; collision mesh filename=/home/nas_main/sibeenkim/work/simtoolreal/assets/urdf/fr3_x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; visual mesh filename=/home/nas_main/sibeenkim/work/simtoolreal/assets/urdf/fr3_x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
- added link mid_tip, mass 0.00000565; collision mesh filename=/home/nas_main/sibeenkim/work/simtoolreal/assets/urdf/fr3_x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; visual mesh filename=/home/nas_main/sibeenkim/work/simtoolreal/assets/urdf/fr3_x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
- added link midback_link1, mass 0.00000002; collision mesh filename=/home/nas_main/sibeenkim/work/simtoolreal/assets/urdf/fr3_x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; visual mesh filename=/home/nas_main/sibeenkim/work/simtoolreal/assets/urdf/fr3_x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
- added link midback_link2, mass 0.00000001; collision mesh filename=/home/nas_main/sibeenkim/work/simtoolreal/assets/urdf/fr3_x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; visual mesh filename=/home/nas_main/sibeenkim/work/simtoolreal/assets/urdf/fr3_x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
- added link pinky_tip, mass 0.00000565; collision mesh filename=/home/nas_main/sibeenkim/work/simtoolreal/assets/urdf/fr3_x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; visual mesh filename=/home/nas_main/sibeenkim/work/simtoolreal/assets/urdf/fr3_x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
- added link pinkyback_link1, mass 0.00000002; collision mesh filename=/home/nas_main/sibeenkim/work/simtoolreal/assets/urdf/fr3_x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; visual mesh filename=/home/nas_main/sibeenkim/work/simtoolreal/assets/urdf/fr3_x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
- added link pinkyback_link2, mass 0.00000001; collision mesh filename=/home/nas_main/sibeenkim/work/simtoolreal/assets/urdf/fr3_x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; visual mesh filename=/home/nas_main/sibeenkim/work/simtoolreal/assets/urdf/fr3_x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
- added link ring_tip, mass 0.00000565; collision mesh filename=/home/nas_main/sibeenkim/work/simtoolreal/assets/urdf/fr3_x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; visual mesh filename=/home/nas_main/sibeenkim/work/simtoolreal/assets/urdf/fr3_x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
- added link ringback_link1, mass 0.00000002; collision mesh filename=/home/nas_main/sibeenkim/work/simtoolreal/assets/urdf/fr3_x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; visual mesh filename=/home/nas_main/sibeenkim/work/simtoolreal/assets/urdf/fr3_x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
- added link ringback_link2, mass 0.00000001; collision mesh filename=/home/nas_main/sibeenkim/work/simtoolreal/assets/urdf/fr3_x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; visual mesh filename=/home/nas_main/sibeenkim/work/simtoolreal/assets/urdf/fr3_x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
- added link thumb_rota_tip, mass 0.00000565; collision mesh filename=/home/nas_main/sibeenkim/work/simtoolreal/assets/urdf/fr3_x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; visual mesh filename=/home/nas_main/sibeenkim/work/simtoolreal/assets/urdf/fr3_x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
- added link thumb_rotaback_link1, mass 0.00000006; collision mesh filename=/home/nas_main/sibeenkim/work/simtoolreal/assets/urdf/fr3_x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; visual mesh filename=/home/nas_main/sibeenkim/work/simtoolreal/assets/urdf/fr3_x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
- added link thumb_rotaback_link2, mass 0.00000004; collision mesh filename=/home/nas_main/sibeenkim/work/simtoolreal/assets/urdf/fr3_x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; visual mesh filename=/home/nas_main/sibeenkim/work/simtoolreal/assets/urdf/fr3_x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
- link index_bend_link: mass None -> 0.068721
- link index_rota_link1: mass None -> 0.06298297
- link index_rota_link2: mass None -> 0.01582395
- link mid_link1: mass None -> 0.06298297
- link mid_link2: mass None -> 0.01582395
- link palm: mass None -> 0.53851506
- link pinky_link1: mass None -> 0.06298297
- link pinky_link2: mass None -> 0.01582395
- link ring_link1: mass None -> 0.06298297
- link ring_link2: mass None -> 0.01582395
- link thumb_bend_link: mass None -> 0.01151453
- link thumb_rota_link1: mass None -> 0.1322853
- link thumb_rota_link2: mass None -> 0.03516871
Joints:
- added joint back_joint: type fixed, parent palm, child back_link, origin xyz=0 0 0.065 rpy=0 0 0, axis 0 0 0
- added joint ee_joint: type fixed, parent palm, child ee_link, origin xyz=0 0 0.065 rpy=0 0 0, axis 0 0 0
- added joint index_rota_joint3: type fixed, parent index_rota_link2, child index_rota_tip, origin xyz=0 0 0.0422482924089424 rpy=0 0 0, axis 0 0 0
- added joint index_rotaback_joint1: type fixed, parent index_rota_link1, child index_rotaback_link1, origin xyz=0 0 0.0557999999999955 rpy=0 0 0, axis 0 0 0
- added joint index_rotaback_joint2: type fixed, parent index_rota_link2, child index_rotaback_link2, origin xyz=0 0 0.0422482924089424 rpy=0 0 0, axis 0 0 0
- added joint mid_joint3: type fixed, parent mid_link2, child mid_tip, origin xyz=0 0 0.042248 rpy=0 0 0, axis 0 0 0
- added joint midback_joint1: type fixed, parent mid_link1, child midback_link1, origin xyz=0 0 0.0558 rpy=0 0 0, axis 0 0 0
- added joint midback_joint2: type fixed, parent mid_link2, child midback_link2, origin xyz=0 0 0.0422482924089416 rpy=0 0 0, axis 0 0 0
- added joint pinky_joint3: type fixed, parent pinky_link2, child pinky_tip, origin xyz=0 0 0.0422482924089405 rpy=0 0 0, axis 0 0 0
- added joint pinkyback_joint1: type fixed, parent pinky_link1, child pinkyback_link1, origin xyz=0 0 0.0558000000000001 rpy=0 0 0, axis 0 0 0
- added joint pinkyback_joint2: type fixed, parent pinky_link2, child pinkyback_link2, origin xyz=0 0 0.0422482924089405 rpy=0 0 0, axis 0 0 0
- added joint ring_joint3: type fixed, parent ring_link2, child ring_tip, origin xyz=0 0 0.0422482924089404 rpy=0 0 0, axis 0 0 0
- added joint ringback_joint1: type fixed, parent ring_link1, child ringback_link1, origin xyz=0 0 0.0558 rpy=0 0 0, axis 0 0 0
- added joint ringback_joint2: type fixed, parent ring_link2, child ringback_link2, origin xyz=0 0 0.0422482924089404 rpy=0 0 0, axis 0 0 0
- added joint thumb_rota_joint3: type fixed, parent thumb_rota_link2, child thumb_rota_tip, origin xyz=0 0.0502276499414863 0 rpy=0 0 0, axis 0 0 0
- added joint thumb_rotaback_joint1: type fixed, parent thumb_rota_link1, child thumb_rotaback_link1, origin xyz=0 0.0553000000000007 0 rpy=0 0 0, axis 0 0 0
- added joint thumb_rotaback_joint2: type fixed, parent thumb_rota_link2, child thumb_rotaback_link2, origin xyz=0 0.0502276499414863 0 rpy=0 0 0, axis 0 0 0
- joint hand_mount: origin xyz=-0.017 -0.017 0.051 rpy=-1.5708 0 -0.7854 -> xyz=-0.017 -0.017 0.051 rpy=-3.1416 -1.5708 0.7854
- joint index_joint0: axis 0 1 0 -> -1 0 0; limit lower=-0.175 upper=0.175 effort=10 velocity=3.14 -> lower=-0.174 upper=0.174 effort=0.4 velocity=14.38; origin xyz=0.0265 -0.0065 0.0899 rpy=0 0 0 -> xyz=0.0065 0.0265 0.0899 rpy=0 0 0
- joint index_joint1: axis 1 0 0 -> 0 1 0; limit lower=0.0 upper=1.92 effort=10 velocity=3.14 -> lower=0 upper=1.919 effort=1.1 velocity=8.63
- joint index_joint2: axis 1 0 0 -> 0 1 0; limit lower=0.0 upper=1.92 effort=10 velocity=3.14 -> lower=0 upper=1.919 effort=0.4 velocity=14.38
- joint middle_joint0: axis 1 0 0 -> 0 1 0; limit lower=0.0 upper=1.92 effort=10 velocity=3.14 -> lower=0 upper=1.919 effort=1.1 velocity=8.63; origin xyz=0.004 -0.0065 0.1082 rpy=0 0 0 -> xyz=0.0065 0.004 0.1082 rpy=0 0 0
- joint middle_joint1: axis 1 0 0 -> 0 1 0; limit lower=0.0 upper=1.92 effort=10 velocity=3.14 -> lower=0 upper=1.919 effort=0.4 velocity=14.38
- joint pinky_joint0: axis 1 0 0 -> 0 1 0; limit lower=0.0 upper=1.92 effort=10 velocity=3.14 -> lower=0 upper=1.919 effort=1.1 velocity=8.63; origin xyz=-0.036 -0.0065 0.1022 rpy=0 0 0 -> xyz=0.0065 -0.036 0.1022 rpy=0 0 0
- joint pinky_joint1: axis 1 0 0 -> 0 1 0; limit lower=0.0 upper=1.92 effort=10 velocity=3.14 -> lower=0 upper=1.919 effort=0.4 velocity=14.38
- joint ring_joint0: axis 1 0 0 -> 0 1 0; limit lower=0.0 upper=1.92 effort=10 velocity=3.14 -> lower=0 upper=1.919 effort=1.1 velocity=8.63; origin xyz=-0.016 -0.0065 0.1052 rpy=0 0 0 -> xyz=0.0065 -0.016 0.1052 rpy=0 0 0
- joint ring_joint1: axis 1 0 0 -> 0 1 0; limit lower=0.0 upper=1.92 effort=10 velocity=3.14 -> lower=0 upper=1.919 effort=0.4 velocity=14.38
- joint thumb_joint0: limit lower=0.0 upper=1.83 effort=10 velocity=3.14 -> lower=0 upper=1.832 effort=1.1 velocity=8.63; origin xyz=0.0228 -0.0095 0.0305 rpy=0 0 0 -> xyz=0.0095 0.0228 0.0305 rpy=0 0 0
- joint thumb_joint1: axis 0 -1 0 -> 1 0 0; limit lower=-1.05 upper=1.57 effort=10 velocity=3.14 -> lower=-0.698 upper=1.57 effort=1.1 velocity=8.63; origin xyz=0.028599 0.0083177 0.00178 rpy=0.2618 0 0.0407 -> xyz=0.0083177 0.028599 -0.00178 rpy=0 0.2618 -0.0407
- joint thumb_joint2: axis 0 -1 0 -> 1 0 0; limit lower=-0.175 upper=1.83 effort=10 velocity=3.14 -> lower=0 upper=1.57 effort=0.4 velocity=14.38; origin xyz=0.0553 0 0 rpy=0 0 0 -> xyz=0 0.0553 0 rpy=0 0 0
