Commit message: fr3_xhand: hand_mount xyz -> hardware-validated LeFranX bracket translation (-0.02616295 -0.02616295 0.042), FK-exact vs do-as-i-do bracket URDF (palm 0.000 mm, tips <0.002 mm)

File: assets/urdf/fr3_xhand_description/fr3_xhand/fr3_xhand.urdf (robot description, URDF)
Before this commit: robot fr3_xhand, 39 links, 38 joints
Joints:
- joint hand_mount: origin xyz=-0.017 -0.017 0.051 rpy=-3.1416 -1.5708 0.7854 -> xyz=-0.02616295 -0.02616295 0.042 rpy=-3.1416 -1.5708 0.7854

Commit message: fr3_xhand: add LeFranX bracket visuals on fr3_link8 (bracket_plate + bracket_base from do-as-i-do DJ MJCF, black, visual-only, link8-frame identity origin)

File: assets/urdf/fr3_xhand_description/fr3_xhand/fr3_xhand.urdf (robot description, URDF)
Before this commit: robot fr3_xhand, 39 links, 38 joints
Links:
- link fr3_link8: geometry visual mesh filename=meshes/bracket_base.obj; visual mesh filename=meshes/bracket_plate.obj

Commit message: fr3_xhand: bracket visuals obj -> stl so the viewer applies the URDF black (0.1 0.1 0.1), OBJ geometry rendered loader-default white in wandb media

File: assets/urdf/fr3_xhand_description/fr3_xhand/fr3_xhand.urdf (robot description, URDF)
Before this commit: robot fr3_xhand, 39 links, 38 joints
Links:
- link fr3_link8: geometry visual mesh filename=meshes/bracket_base.stl; visual mesh filename=meshes/bracket_plate.stl

Commit message: fr3_xhand urdf: mesh paths relative

File: assets/urdf/fr3_xhand_description/fr3_xhand/fr3_xhand.urdf (robot description, URDF)
Before this commit: robot fr3_xhand, 39 links, 38 joints
Links:
- link back_link: geometry collision mesh filename=../xhand1_right/meshes/right_hand_back_link.STL; visual mesh filename=../xhand1_right/meshes/right_hand_back_link.STL
- link ee_link: geometry collision mesh filename=../xhand1_right/meshes/right_hand_ee_link.STL; visual mesh filename=../xhand1_right/meshes/right_hand_ee_link.STL
- link fr3_link0: geometry collision mesh filename=../fr3/meshes/collision/link0.stl; visual mesh filename=../fr3/meshes/visual/link0.stl
- link fr3_link1: geometry collision mesh filename=../fr3/meshes/collision/link1.stl; visual mesh filename=../fr3/meshes/visual/link1.stl
- link fr3_link2: geometry collision mesh filename=../fr3/meshes/collision/link2.stl; visual mesh filename=../fr3/meshes/visual/link2.stl
- link fr3_link3: geometry collision mesh filename=../fr3/meshes/collision/link3.stl; visual mesh filename=../fr3/meshes/visual/link3.stl
- link fr3_link4: geometry collision mesh filename=../fr3/meshes/collision/link4.stl; visual mesh filename=../fr3/meshes/visual/link4.stl
- link fr3_link5: geometry collision mesh filename=../fr3/meshes/collision/link5.stl; visual mesh filename=../fr3/meshes/visual/link5.stl
- link fr3_link6: geometry collision mesh filename=../fr3/meshes/collision/link6.stl; visual mesh filename=../fr3/meshes/visual/link6.stl
- link fr3_link7: geometry collision mesh filename=../fr3/meshes/collision/link7.stl; visual mesh filename=../fr3/meshes/visual/link7.stl
- link index_bend_link: geometry collision mesh filename=../xhand1_right/meshes/right_hand_index_bend_link.STL; visual mesh filename=../xhand1_right/meshes/right_hand_index_bend_link.STL
- link index_rota_link1: geometry collision mesh filename=../xhand1_right/meshes/right_hand_index_rota_link1.STL; visual mesh filename=../xhand1_right/meshes/right_hand_index_rota_link1.STL
- link index_rota_link2: geometry collision mesh filename=../xhand1_right/meshes/right_hand_index_rota_link2.STL; visual mesh filename=../xhand1_right/meshes/right_hand_index_rota_link2.STL
- link index_rota_tip: geometry collision mesh filename=../xhand1_right/meshes/right_hand_index_rota_tip.STL; visual mesh filename=../xhand1_right/meshes/right_hand_index_rota_tip.STL
- link index_rotaback_link1: geometry collision mesh filename=../xhand1_right/meshes/right_hand_index_rotaback_link1.STL; visual mesh filename=../xhand1_right/meshes/right_hand_index_rotaback_link1.STL
- link index_rotaback_link2: geometry collision mesh filename=../xhand1_right/meshes/right_hand_index_rotaback_link2.STL; visual mesh filename=../xhand1_right/meshes/right_hand_index_rotaback_link2.STL
- link mid_link1: geometry collision mesh filename=../xhand1_right/meshes/right_hand_mid_link1.STL; visual mesh filename=../xhand1_right/meshes/right_hand_mid_link1.STL
- link mid_link2: geometry collision mesh filename=../xhand1_right/meshes/right_hand_mid_link2.STL; visual mesh filename=../xhand1_right/meshes/right_hand_mid_link2.STL
- link mid_tip: geometry collision mesh filename=../xhand1_right/meshes/right_hand_mid_tip.STL; visual mesh filename=../xhand1_right/meshes/right_hand_mid_tip.STL
- link midback_link1: geometry collision mesh filename=../xhand1_right/meshes/right_hand_midback_link1.STL; visual mesh filename=../xhand1_right/meshes/right_hand_midback_link1.STL
- link midback_link2: geometry collision mesh filename=../xhand1_right/meshes/right_hand_midback_link2.STL; visual mesh filename=../xhand1_right/meshes/right_hand_midback_link2.STL
- link palm: geometry collision mesh filename=../xhand1_right/meshes/right_hand_link.STL; visual mesh filename=../xhand1_right/meshes/right_hand_link.STL
- link pinky_link1: geometry collision mesh filename=../xhand1_right/meshes/right_hand_pinky_link1.STL; visual mesh filename=../xhand1_right/meshes/right_hand_pinky_link1.STL
- link pinky_link2: geometry collision mesh filename=../xhand1_right/meshes/right_hand_pinky_link2.STL; visual mesh filename=../xhand1_right/meshes/right_hand_pinky_link2.STL
- link pinky_tip: geometry collision mesh filename=../xhand1_right/meshes/right_hand_pinky_tip.STL; visual mesh filename=../xhand1_right/meshes/right_hand_pinky_tip.STL
- link pinkyback_link1: geometry collision mesh filename=../xhand1_right/meshes/right_hand_pinkyback_link1.STL; visual mesh filename=../xhand1_right/meshes/right_hand_pinkyback_link1.STL
- link pinkyback_link2: geometry collision mesh filename=../xhand1_right/meshes/right_hand_pinkyback_link2.STL; visual mesh filename=../xhand1_right/meshes/right_hand_pinkyback_link2.STL
- link ring_link1: geometry collision mesh filename=../xhand1_right/meshes/right_hand_ring_link1.STL; visual mesh filename=../xhand1_right/meshes/right_hand_ring_link1.STL
- link ring_link2: geometry collision mesh filename=../xhand1_right/meshes/right_hand_ring_link2.STL; visual mesh filename=../xhand1_right/meshes/right_hand_ring_link2.STL
- link ring_tip: geometry collision mesh filename=../xhand1_right/meshes/right_hand_ring_tip.STL; visual mesh filename=../xhand1_right/meshes/right_hand_ring_tip.STL
- link ringback_link1: geometry collision mesh filename=../xhand1_right/meshes/right_hand_ringback_link1.STL; visual mesh filename=../xhand1_right/meshes/right_hand_ringback_link1.STL
- link ringback_link2: geometry collision mesh filename=../xhand1_right/meshes/right_hand_ringback_link2.STL; visual mesh filename=../xhand1_right/meshes/right_hand_ringback_link2.STL
- link thumb_bend_link: geometry collision mesh filename=../xhand1_right/meshes/right_hand_thumb_bend_link.STL; visual mesh filename=../xhand1_right/meshes/right_hand_thumb_bend_link.STL
- link thumb_rota_link1: geometry collision mesh filename=../xhand1_right/meshes/right_hand_thumb_rota_link1.STL; visual mesh filename=../xhand1_right/meshes/right_hand_thumb_rota_link1.STL
- link thumb_rota_link2: geometry collision mesh filename=../xhand1_right/meshes/right_hand_thumb_rota_link2.STL; visual mesh filename=../xhand1_right/meshes/right_hand_thumb_rota_link2.STL
- link thumb_rota_tip: geometry collision mesh filename=../xhand1_right/meshes/right_hand_thumb_rota_tip.STL; visual mesh filename=../xhand1_right/meshes/right_hand_thumb_rota_tip.STL
- link thumb_rotaback_link1: geometry collision mesh filename=../xhand1_right/meshes/right_hand_thumb_rotaback_link1.STL; visual mesh filename=../xhand1_right/meshes/right_hand_thumb_rotaback_link1.STL
- link thumb_rotaback_link2: geometry collision mesh filename=../xhand1_right/meshes/right_hand_thumb_rotaback_link2.STL; visual mesh filename=../xhand1_right/meshes/right_hand_thumb_rotaback_link2.STL

Commit message: fr3+xhand: vendor physics set, and the arm/hand gain sweep profiles
Every value comes from franka_description 2.8.1 fr3v2 or the FCI control
parameter tables. None of it is our own measurement.

  scene_utils  robot base (0.0, 0.8, 0.0) -> (0.0, 0.48, 0.53), session 027
               arm actuator now takes armature and friction
  robots.py    reset pose -> [-90, 15, 0, -115, 0, 135, -45] deg
               arm_armature = motor_inertia * gear_ratio^2, fr3v2/dynamics.yaml
               arm_friction 0.2 flat, same file
               hand_armature 0.001 -> 0; vendor URDF, RoboVerse and ConTrack
               all set none, and the hand is direct drive so there is no
               gear ratio to square
  urdf         arm link inertials, FER 16.691901 kg -> fr3v2 15.907822 kg
               arm joint limits -> FCI control parameters
               fr3_link8 gains a 0.218 kg inertial; it had none, so the
               bracket weighed nothing

The hand URDF already carried the vendor efforts, velocities and joint
limits, so it is untouched.

Eight sweep profiles, fr3-xhand-{a1..a4}{h1,h2}. a1 and a2 take kp from
franka_ros2 controllers.yaml, a3 and a4 from IsaacLab FRANKA_PANDA_HIGH_PD_CFG.
kd is either as that source ships it or 2*sqrt(kp*armature). h1 is RoboVerse
flat 0.1, h2 is 2*sqrt(kp*M_ii) per joint. fr3-xhand-adapter and fr3-xhand
keep their existing gains as a3h1.

File: assets/urdf/fr3_xhand_description/fr3_xhand/fr3_xhand.urdf (robot description, URDF)
Before this commit: robot fr3_xhand, 39 links, 38 joints
Links:
- link fr3_link0: mass 0.629769 -> 2.396600
- link fr3_link1: mass 4.970684 -> 2.437700
- link fr3_link2: mass 0.646926 -> 2.237500
- link fr3_link3: mass 3.228604 -> 2.193082
- link fr3_link4: mass 3.587895 -> 2.181537
- link fr3_link5: mass 1.225946 -> 2.186881
- link fr3_link6: mass 1.666555 -> 1.579681
- link fr3_link7: mass 0.735522 -> 0.694841
- link fr3_link8: mass None -> 0.218000
Joints:
- joint fr3_joint1: limit lower=-2.7437 upper=2.7437 effort=87 velocity=2.62 -> lower=-2.9007400166666666 upper=2.9007400166666666 effort=87 velocity=2.62
- joint fr3_joint2: limit lower=-1.7837 upper=1.7837 effort=87 velocity=2.62 -> lower=-1.8360900166666667 upper=1.8360900166666667 effort=87 velocity=2.62
- joint fr3_joint3: limit lower=-2.9007 upper=2.9007 effort=87 velocity=2.62 -> lower=-2.9007400166666666 upper=2.9007400166666666 effort=87 velocity=2.62
- joint fr3_joint4: limit lower=-3.0421 upper=-0.1518 effort=87 velocity=2.62 -> lower=-3.077020016666667 upper=-0.11693708333333333 effort=87 velocity=2.62
- joint fr3_joint5: limit lower=-2.8065 upper=2.8065 effort=12 velocity=5.26 -> lower=-2.87630335 upper=2.87630335 effort=12 velocity=5.26
- joint fr3_joint6: limit lower=0.5445 upper=4.5169 effort=12 velocity=4.18 -> lower=0.43982265 upper=4.62163335 effort=12 velocity=4.18
- joint fr3_joint7: limit lower=-3.0159 upper=3.0159 effort=12 velocity=5.26 -> lower=-3.05083335 upper=3.05083335 effort=12 velocity=5.26

File: assets/urdf/fr3_xhand_description/fr3_xhand/fr3_xhand_noadapter.urdf (robot description, URDF)
Before this commit: robot fr3_xhand, 39 links, 38 joints
Links:
- link fr3_link0: mass 0.629769 -> 2.396600
- link fr3_link1: mass 4.970684 -> 2.437700
- link fr3_link2: mass 0.646926 -> 2.237500
- link fr3_link3: mass 3.228604 -> 2.193082
- link fr3_link4: mass 3.587895 -> 2.181537
- link fr3_link5: mass 1.225946 -> 2.186881
- link fr3_link6: mass 1.666555 -> 1.579681
- link fr3_link7: mass 0.735522 -> 0.694841
Joints:
- joint fr3_joint1: limit lower=-2.7437 upper=2.7437 effort=87 velocity=2.62 -> lower=-2.9007400166666666 upper=2.9007400166666666 effort=87 velocity=2.62
- joint fr3_joint2: limit lower=-1.7837 upper=1.7837 effort=87 velocity=2.62 -> lower=-1.8360900166666667 upper=1.8360900166666667 effort=87 velocity=2.62
- joint fr3_joint3: limit lower=-2.9007 upper=2.9007 effort=87 velocity=2.62 -> lower=-2.9007400166666666 upper=2.9007400166666666 effort=87 velocity=2.62
- joint fr3_joint4: limit lower=-3.0421 upper=-0.1518 effort=87 velocity=2.62 -> lower=-3.077020016666667 upper=-0.11693708333333333 effort=87 velocity=2.62
- joint fr3_joint5: limit lower=-2.8065 upper=2.8065 effort=12 velocity=5.26 -> lower=-2.87630335 upper=2.87630335 effort=12 velocity=5.26
- joint fr3_joint6: limit lower=0.5445 upper=4.5169 effort=12 velocity=4.18 -> lower=0.43982265 upper=4.62163335 effort=12 velocity=4.18
- joint fr3_joint7: limit lower=-3.0159 upper=3.0159 effort=12 velocity=5.26 -> lower=-3.05083335 upper=3.05083335 effort=12 velocity=5.26
