Commit message: rename hand links and joints

File: assets/urdf/fr3_xhand_description/fr3_xhand/fr3_xhand.urdf (robot description, URDF)
Before this commit: robot fr3_xhand, 39 links, 38 joints
Links:
- removed link right_hand_back_link
- removed link right_hand_ee_link
- removed link right_hand_index_bend_link
- removed link right_hand_index_rota_link1
- removed link right_hand_index_rota_link2
- removed link right_hand_index_rota_tip
- removed link right_hand_index_rotaback_link1
- removed link right_hand_index_rotaback_link2
- removed link right_hand_link
- removed link right_hand_mid_link1
- removed link right_hand_mid_link2
- removed link right_hand_mid_tip
- removed link right_hand_midback_link1
- removed link right_hand_midback_link2
- removed link right_hand_pinky_link1
- removed link right_hand_pinky_link2
- removed link right_hand_pinky_tip
- removed link right_hand_pinkyback_link1
- removed link right_hand_pinkyback_link2
- removed link right_hand_ring_link1
- removed link right_hand_ring_link2
- removed link right_hand_ring_tip
- removed link right_hand_ringback_link1
- removed link right_hand_ringback_link2
- removed link right_hand_thumb_bend_link
- removed link right_hand_thumb_rota_link1
- removed link right_hand_thumb_rota_link2
- removed link right_hand_thumb_rota_tip
- removed link right_hand_thumb_rotaback_link1
- removed link right_hand_thumb_rotaback_link2
- added link back_link, mass 0.00000002; collision mesh filename=../xhand1_right/meshes/right_hand_back_link.STL; visual mesh filename=../xhand1_right/meshes/right_hand_back_link.STL
- added link ee_link, mass 0.00000565; collision mesh filename=../xhand1_right/meshes/right_hand_ee_link.STL; visual mesh filename=../xhand1_right/meshes/right_hand_ee_link.STL
- added link index_bend_link, mass 0.068721; collision mesh filename=../xhand1_right/meshes/right_hand_index_bend_link.STL; visual mesh filename=../xhand1_right/meshes/right_hand_index_bend_link.STL
- added link index_rota_link1, mass 0.06298297; collision mesh filename=../xhand1_right/meshes/right_hand_index_rota_link1.STL; visual mesh filename=../xhand1_right/meshes/right_hand_index_rota_link1.STL
- added link index_rota_link2, mass 0.01582395; collision mesh filename=../xhand1_right/meshes/right_hand_index_rota_link2.STL; visual mesh filename=../xhand1_right/meshes/right_hand_index_rota_link2.STL
- added link index_rota_tip, mass 0.00000565; collision mesh filename=../xhand1_right/meshes/right_hand_index_rota_tip.STL; visual mesh filename=../xhand1_right/meshes/right_hand_index_rota_tip.STL
- added link index_rotaback_link1, mass 0.00000002; collision mesh filename=../xhand1_right/meshes/right_hand_index_rotaback_link1.STL; visual mesh filename=../xhand1_right/meshes/right_hand_index_rotaback_link1.STL
- added link index_rotaback_link2, mass 0.00000001; collision mesh filename=../xhand1_right/meshes/right_hand_index_rotaback_link2.STL; visual mesh filename=../xhand1_right/meshes/right_hand_index_rotaback_link2.STL
- added link mid_link1, mass 0.06298297; collision mesh filename=../xhand1_right/meshes/right_hand_mid_link1.STL; visual mesh filename=../xhand1_right/meshes/right_hand_mid_link1.STL
- added link mid_link2, mass 0.01582395; collision mesh filename=../xhand1_right/meshes/right_hand_mid_link2.STL; visual mesh filename=../xhand1_right/meshes/right_hand_mid_link2.STL
- added link mid_tip, mass 0.00000565; collision mesh filename=../xhand1_right/meshes/right_hand_mid_tip.STL; visual mesh filename=../xhand1_right/meshes/right_hand_mid_tip.STL
- added link midback_link1, mass 0.00000002; collision mesh filename=../xhand1_right/meshes/right_hand_midback_link1.STL; visual mesh filename=../xhand1_right/meshes/right_hand_midback_link1.STL
- added link midback_link2, mass 0.00000001; collision mesh filename=../xhand1_right/meshes/right_hand_midback_link2.STL; visual mesh filename=../xhand1_right/meshes/right_hand_midback_link2.STL
- added link palm, mass 0.53851506; collision mesh filename=../xhand1_right/meshes/right_hand_link.STL; visual mesh filename=../xhand1_right/meshes/right_hand_link.STL
- added link pinky_link1, mass 0.06298297; collision mesh filename=../xhand1_right/meshes/right_hand_pinky_link1.STL; visual mesh filename=../xhand1_right/meshes/right_hand_pinky_link1.STL
- added link pinky_link2, mass 0.01582395; collision mesh filename=../xhand1_right/meshes/right_hand_pinky_link2.STL; visual mesh filename=../xhand1_right/meshes/right_hand_pinky_link2.STL
- added link pinky_tip, mass 0.00000565; collision mesh filename=../xhand1_right/meshes/right_hand_pinky_tip.STL; visual mesh filename=../xhand1_right/meshes/right_hand_pinky_tip.STL
- added link pinkyback_link1, mass 0.00000002; collision mesh filename=../xhand1_right/meshes/right_hand_pinkyback_link1.STL; visual mesh filename=../xhand1_right/meshes/right_hand_pinkyback_link1.STL
- added link pinkyback_link2, mass 0.00000001; collision mesh filename=../xhand1_right/meshes/right_hand_pinkyback_link2.STL; visual mesh filename=../xhand1_right/meshes/right_hand_pinkyback_link2.STL
- added link ring_link1, mass 0.06298297; collision mesh filename=../xhand1_right/meshes/right_hand_ring_link1.STL; visual mesh filename=../xhand1_right/meshes/right_hand_ring_link1.STL
- added link ring_link2, mass 0.01582395; collision mesh filename=../xhand1_right/meshes/right_hand_ring_link2.STL; visual mesh filename=../xhand1_right/meshes/right_hand_ring_link2.STL
- added link ring_tip, mass 0.00000565; collision mesh filename=../xhand1_right/meshes/right_hand_ring_tip.STL; visual mesh filename=../xhand1_right/meshes/right_hand_ring_tip.STL
- added link ringback_link1, mass 0.00000002; collision mesh filename=../xhand1_right/meshes/right_hand_ringback_link1.STL; visual mesh filename=../xhand1_right/meshes/right_hand_ringback_link1.STL
- added link ringback_link2, mass 0.00000001; collision mesh filename=../xhand1_right/meshes/right_hand_ringback_link2.STL; visual mesh filename=../xhand1_right/meshes/right_hand_ringback_link2.STL
- added link thumb_bend_link, mass 0.01151453; collision mesh filename=../xhand1_right/meshes/right_hand_thumb_bend_link.STL; visual mesh filename=../xhand1_right/meshes/right_hand_thumb_bend_link.STL
- added link thumb_rota_link1, mass 0.1322853; collision mesh filename=../xhand1_right/meshes/right_hand_thumb_rota_link1.STL; visual mesh filename=../xhand1_right/meshes/right_hand_thumb_rota_link1.STL
- added link thumb_rota_link2, mass 0.03516871; collision mesh filename=../xhand1_right/meshes/right_hand_thumb_rota_link2.STL; visual mesh filename=../xhand1_right/meshes/right_hand_thumb_rota_link2.STL
- added link thumb_rota_tip, mass 0.00000565; collision mesh filename=../xhand1_right/meshes/right_hand_thumb_rota_tip.STL; visual mesh filename=../xhand1_right/meshes/right_hand_thumb_rota_tip.STL
- added link thumb_rotaback_link1, mass 0.00000006; collision mesh filename=../xhand1_right/meshes/right_hand_thumb_rotaback_link1.STL; visual mesh filename=../xhand1_right/meshes/right_hand_thumb_rotaback_link1.STL
- added link thumb_rotaback_link2, mass 0.00000004; collision mesh filename=../xhand1_right/meshes/right_hand_thumb_rotaback_link2.STL; visual mesh filename=../xhand1_right/meshes/right_hand_thumb_rotaback_link2.STL
Joints:
- removed joint right_hand_back_joint
- removed joint right_hand_ee_joint
- removed joint right_hand_index_bend_joint
- removed joint right_hand_index_joint1
- removed joint right_hand_index_joint2
- removed joint right_hand_index_rota_joint3
- removed joint right_hand_index_rotaback_joint1
- removed joint right_hand_index_rotaback_joint2
- removed joint right_hand_mid_joint1
- removed joint right_hand_mid_joint2
- removed joint right_hand_mid_joint3
- removed joint right_hand_midback_joint1
- removed joint right_hand_midback_joint2
- removed joint right_hand_pinky_joint1
- removed joint right_hand_pinky_joint2
- removed joint right_hand_pinky_joint3
- removed joint right_hand_pinkyback_joint1
- removed joint right_hand_pinkyback_joint2
- removed joint right_hand_ring_joint1
- removed joint right_hand_ring_joint2
- removed joint right_hand_ring_joint3
- removed joint right_hand_ringback_joint1
- removed joint right_hand_ringback_joint2
- removed joint right_hand_thumb_bend_joint
- removed joint right_hand_thumb_rota_joint1
- removed joint right_hand_thumb_rota_joint2
- removed joint right_hand_thumb_rota_joint3
- removed joint right_hand_thumb_rotaback_joint1
- removed joint right_hand_thumb_rotaback_joint2
- added joint back_joint: type fixed, parent palm, child back_link, origin xyz=0 0 0.065 rpy=0 0 0, axis 0 0 0
- added joint ee_joint: type fixed, parent palm, child ee_link, origin xyz=0 0 0.065 rpy=0 0 0, axis 0 0 0
- added joint index_joint0: type revolute, parent palm, child index_bend_link, origin xyz=0.0065 0.0265 0.0899 rpy=0 0 0, axis -1 0 0, limit lower=-0.174 upper=0.174 effort=0.4 velocity=14.38
- added joint index_joint1: type revolute, parent index_bend_link, child index_rota_link1, origin xyz=0 0 0.0178 rpy=0 0 0, axis 0 1 0, limit lower=0 upper=1.919 effort=1.1 velocity=8.63
- added joint index_joint2: type revolute, parent index_rota_link1, child index_rota_link2, origin xyz=0 0 0.0558 rpy=0 0 0, axis 0 1 0, limit lower=0 upper=1.919 effort=0.4 velocity=14.38
- added joint index_rota_joint3: type fixed, parent index_rota_link2, child index_rota_tip, origin xyz=0 0 0.0422482924089424 rpy=0 0 0, axis 0 0 0
- added joint index_rotaback_joint1: type fixed, parent index_rota_link1, child index_rotaback_link1, origin xyz=0 0 0.0557999999999955 rpy=0 0 0, axis 0 0 0
- added joint index_rotaback_joint2: type fixed, parent index_rota_link2, child index_rotaback_link2, origin xyz=0 0 0.0422482924089424 rpy=0 0 0, axis 0 0 0
- added joint mid_joint3: type fixed, parent mid_link2, child mid_tip, origin xyz=0 0 0.042248 rpy=0 0 0, axis 0 0 0
- added joint midback_joint1: type fixed, parent mid_link1, child midback_link1, origin xyz=0 0 0.0558 rpy=0 0 0, axis 0 0 0
- added joint midback_joint2: type fixed, parent mid_link2, child midback_link2, origin xyz=0 0 0.0422482924089416 rpy=0 0 0, axis 0 0 0
- added joint middle_joint0: type revolute, parent palm, child mid_link1, origin xyz=0.0065 0.004 0.1082 rpy=0 0 0, axis 0 1 0, limit lower=0 upper=1.919 effort=1.1 velocity=8.63
- added joint middle_joint1: type revolute, parent mid_link1, child mid_link2, origin xyz=0 0 0.0558 rpy=0 0 0, axis 0 1 0, limit lower=0 upper=1.919 effort=0.4 velocity=14.38
- added joint pinky_joint0: type revolute, parent palm, child pinky_link1, origin xyz=0.0065 -0.036 0.1022 rpy=0 0 0, axis 0 1 0, limit lower=0 upper=1.919 effort=1.1 velocity=8.63
- added joint pinky_joint1: type revolute, parent pinky_link1, child pinky_link2, origin xyz=0 0 0.0558 rpy=0 0 0, axis 0 1 0, limit lower=0 upper=1.919 effort=0.4 velocity=14.38
- added joint pinky_joint3: type fixed, parent pinky_link2, child pinky_tip, origin xyz=0 0 0.0422482924089405 rpy=0 0 0, axis 0 0 0
- added joint pinkyback_joint1: type fixed, parent pinky_link1, child pinkyback_link1, origin xyz=0 0 0.0558000000000001 rpy=0 0 0, axis 0 0 0
- added joint pinkyback_joint2: type fixed, parent pinky_link2, child pinkyback_link2, origin xyz=0 0 0.0422482924089405 rpy=0 0 0, axis 0 0 0
- added joint ring_joint0: type revolute, parent palm, child ring_link1, origin xyz=0.0065 -0.016 0.1052 rpy=0 0 0, axis 0 1 0, limit lower=0 upper=1.919 effort=1.1 velocity=8.63
- added joint ring_joint1: type revolute, parent ring_link1, child ring_link2, origin xyz=0 0 0.0558 rpy=0 0 0, axis 0 1 0, limit lower=0 upper=1.919 effort=0.4 velocity=14.38
- added joint ring_joint3: type fixed, parent ring_link2, child ring_tip, origin xyz=0 0 0.0422482924089404 rpy=0 0 0, axis 0 0 0
- added joint ringback_joint1: type fixed, parent ring_link1, child ringback_link1, origin xyz=0 0 0.0558 rpy=0 0 0, axis 0 0 0
- added joint ringback_joint2: type fixed, parent ring_link2, child ringback_link2, origin xyz=0 0 0.0422482924089404 rpy=0 0 0, axis 0 0 0
- added joint thumb_joint0: type revolute, parent palm, child thumb_bend_link, origin xyz=0.0095 0.0228 0.0305 rpy=0 0 0, axis 0 0 -1, limit lower=0 upper=1.832 effort=1.1 velocity=8.63
- added joint thumb_joint1: type revolute, parent thumb_bend_link, child thumb_rota_link1, origin xyz=0.0083177 0.028599 -0.00178 rpy=0 0.2618 -0.0407, axis 1 0 0, limit lower=-0.698 upper=1.57 effort=1.1 velocity=8.63
- added joint thumb_joint2: type revolute, parent thumb_rota_link1, child thumb_rota_link2, origin xyz=0 0.0553 0 rpy=0 0 0, axis 1 0 0, limit lower=0 upper=1.57 effort=0.4 velocity=14.38
- added joint thumb_rota_joint3: type fixed, parent thumb_rota_link2, child thumb_rota_tip, origin xyz=0 0.0502276499414863 0 rpy=0 0 0, axis 0 0 0
- added joint thumb_rotaback_joint1: type fixed, parent thumb_rota_link1, child thumb_rotaback_link1, origin xyz=0 0.0553000000000007 0 rpy=0 0 0, axis 0 0 0
- added joint thumb_rotaback_joint2: type fixed, parent thumb_rota_link2, child thumb_rotaback_link2, origin xyz=0 0.0502276499414863 0 rpy=0 0 0, axis 0 0 0
- joint hand_mount: child right_hand_link -> palm
