Commit message: fr3-xhand: straight mount + 23.5mm RobotEra adapter (visual, black), deploy home pose [0,0,0,-135,0,225,-45]deg, relative mesh paths

File: assets/urdf/fr3_xhand_description/fr3_xhand/fr3_xhand_noadapter.urdf (robot description, URDF)
Before this commit: robot fr3_xhand, 39 links, 38 joints
Links:
- added link adapter_link; visual mesh filename=../adapter/robotera_adapter.stl
- link back_link: geometry collision mesh filename=../xhand1_right/meshes/right_hand_back_link.STL; visual mesh filename=../xhand1_right/meshes/right_hand_back_link.STL
- link ee_link: geometry collision mesh filename=../xhand1_right/meshes/right_hand_ee_link.STL; visual mesh filename=../xhand1_right/meshes/right_hand_ee_link.STL
- link fr3_link0: geometry collision mesh filename=../fr3/meshes/collision/link0.stl; visual mesh filename=../fr3/meshes/visual/link0.stl
- link fr3_link1: geometry collision mesh filename=../fr3/meshes/collision/link1.stl; visual mesh filename=../fr3/meshes/visual/link1.stl
- link fr3_link2: geometry collision mesh filename=../fr3/meshes/collision/link2.stl; visual mesh filename=../fr3/meshes/visual/link2.stl
- link fr3_link3: geometry collision mesh filename=../fr3/meshes/collision/link3.stl; visual mesh filename=../fr3/meshes/visual/link3.stl
- link fr3_link4: geometry collision mesh filename=../fr3/meshes/collision/link4.stl; visual mesh filename=../fr3/meshes/visual/link4.stl
- link fr3_link5: geometry collision mesh filename=../fr3/meshes/collision/link5.stl; visual mesh filename=../fr3/meshes/visual/link5.stl
- link fr3_link6: geometry collision mesh filename=../fr3/meshes/collision/link6.stl; visual mesh filename=../fr3/meshes/visual/link6.stl
- link fr3_link7: geometry collision mesh filename=../fr3/meshes/collision/link7.stl; visual mesh filename=../fr3/meshes/visual/link7.stl
- link index_bend_link: geometry collision mesh filename=../xhand1_right/meshes/right_hand_index_bend_link.STL; visual mesh filename=../xhand1_right/meshes/right_hand_index_bend_link.STL
- link index_rota_link1: geometry collision mesh filename=../xhand1_right/meshes/right_hand_index_rota_link1.STL; visual mesh filename=../xhand1_right/meshes/right_hand_index_rota_link1.STL
- link index_rota_link2: geometry collision mesh filename=../xhand1_right/meshes/right_hand_index_rota_link2.STL; visual mesh filename=../xhand1_right/meshes/right_hand_index_rota_link2.STL
- link index_rota_tip: geometry collision mesh filename=../xhand1_right/meshes/right_hand_index_rota_tip.STL; visual mesh filename=../xhand1_right/meshes/right_hand_index_rota_tip.STL
- link index_rotaback_link1: geometry collision mesh filename=../xhand1_right/meshes/right_hand_index_rotaback_link1.STL; visual mesh filename=../xhand1_right/meshes/right_hand_index_rotaback_link1.STL
- link index_rotaback_link2: geometry collision mesh filename=../xhand1_right/meshes/right_hand_index_rotaback_link2.STL; visual mesh filename=../xhand1_right/meshes/right_hand_index_rotaback_link2.STL
- link mid_link1: geometry collision mesh filename=../xhand1_right/meshes/right_hand_mid_link1.STL; visual mesh filename=../xhand1_right/meshes/right_hand_mid_link1.STL
- link mid_link2: geometry collision mesh filename=../xhand1_right/meshes/right_hand_mid_link2.STL; visual mesh filename=../xhand1_right/meshes/right_hand_mid_link2.STL
- link mid_tip: geometry collision mesh filename=../xhand1_right/meshes/right_hand_mid_tip.STL; visual mesh filename=../xhand1_right/meshes/right_hand_mid_tip.STL
- link midback_link1: geometry collision mesh filename=../xhand1_right/meshes/right_hand_midback_link1.STL; visual mesh filename=../xhand1_right/meshes/right_hand_midback_link1.STL
- link midback_link2: geometry collision mesh filename=../xhand1_right/meshes/right_hand_midback_link2.STL; visual mesh filename=../xhand1_right/meshes/right_hand_midback_link2.STL
- link palm: geometry collision mesh filename=../xhand1_right/meshes/right_hand_link.STL; visual mesh filename=../xhand1_right/meshes/right_hand_link.STL
- link pinky_link1: geometry collision mesh filename=../xhand1_right/meshes/right_hand_pinky_link1.STL; visual mesh filename=../xhand1_right/meshes/right_hand_pinky_link1.STL
- link pinky_link2: geometry collision mesh filename=../xhand1_right/meshes/right_hand_pinky_link2.STL; visual mesh filename=../xhand1_right/meshes/right_hand_pinky_link2.STL
- link pinky_tip: geometry collision mesh filename=../xhand1_right/meshes/right_hand_pinky_tip.STL; visual mesh filename=../xhand1_right/meshes/right_hand_pinky_tip.STL
- link pinkyback_link1: geometry collision mesh filename=../xhand1_right/meshes/right_hand_pinkyback_link1.STL; visual mesh filename=../xhand1_right/meshes/right_hand_pinkyback_link1.STL
- link pinkyback_link2: geometry collision mesh filename=../xhand1_right/meshes/right_hand_pinkyback_link2.STL; visual mesh filename=../xhand1_right/meshes/right_hand_pinkyback_link2.STL
- link ring_link1: geometry collision mesh filename=../xhand1_right/meshes/right_hand_ring_link1.STL; visual mesh filename=../xhand1_right/meshes/right_hand_ring_link1.STL
- link ring_link2: geometry collision mesh filename=../xhand1_right/meshes/right_hand_ring_link2.STL; visual mesh filename=../xhand1_right/meshes/right_hand_ring_link2.STL
- link ring_tip: geometry collision mesh filename=../xhand1_right/meshes/right_hand_ring_tip.STL; visual mesh filename=../xhand1_right/meshes/right_hand_ring_tip.STL
- link ringback_link1: geometry collision mesh filename=../xhand1_right/meshes/right_hand_ringback_link1.STL; visual mesh filename=../xhand1_right/meshes/right_hand_ringback_link1.STL
- link ringback_link2: geometry collision mesh filename=../xhand1_right/meshes/right_hand_ringback_link2.STL; visual mesh filename=../xhand1_right/meshes/right_hand_ringback_link2.STL
- link thumb_bend_link: geometry collision mesh filename=../xhand1_right/meshes/right_hand_thumb_bend_link.STL; visual mesh filename=../xhand1_right/meshes/right_hand_thumb_bend_link.STL
- link thumb_rota_link1: geometry collision mesh filename=../xhand1_right/meshes/right_hand_thumb_rota_link1.STL; visual mesh filename=../xhand1_right/meshes/right_hand_thumb_rota_link1.STL
- link thumb_rota_link2: geometry collision mesh filename=../xhand1_right/meshes/right_hand_thumb_rota_link2.STL; visual mesh filename=../xhand1_right/meshes/right_hand_thumb_rota_link2.STL
- link thumb_rota_tip: geometry collision mesh filename=../xhand1_right/meshes/right_hand_thumb_rota_tip.STL; visual mesh filename=../xhand1_right/meshes/right_hand_thumb_rota_tip.STL
- link thumb_rotaback_link1: geometry collision mesh filename=../xhand1_right/meshes/right_hand_thumb_rotaback_link1.STL; visual mesh filename=../xhand1_right/meshes/right_hand_thumb_rotaback_link1.STL
- link thumb_rotaback_link2: geometry collision mesh filename=../xhand1_right/meshes/right_hand_thumb_rotaback_link2.STL; visual mesh filename=../xhand1_right/meshes/right_hand_thumb_rotaback_link2.STL
Joints:
- added joint adapter_joint: type fixed, parent fr3_link8, child adapter_link, origin xyz=0 0 0.0235 rpy=0 0 0
- joint hand_mount: parent fr3_link8 -> adapter_link
